File: PowerSupply/Schematic/PowerSupply.kicad_sch (KiCad schematic)
At the start: 193 parts, among them Q1 BC337, Q10 IRLIZ44N, Q11 IRF4905, Q12 IRLIZ44N, Q13 BC337, Q14 BC328, Q15 IRLIZ44N, Q16 BC337, Q2 BC328, Q3 BC337, Q33 BC337, Q34 BC337, Q35 BC337, Q36 BC337, Q37 BC337, Q38 BC328, Q39 BC337, Q4 BC328, Q40 BC328, Q41 BC337, Q42 BC337, Q43 BC337, Q44 BC337, Q45 BC337, Q46 BC337, Q47 BC328, Q48 BC328, Q49 BC337, Q5 BC337, Q50 BD910, Q51 BD909, Q52 IRLIZ44N, Q6 BC328, Q7 BC337, Q8 BC328, Q9 IRF4905, T1 Transformer_1P_2S, U1 TL494, U2 PC817

Commit message: Add files via upload
Parts:
- removed R114: 100, symbol Device:R
- R111: value 10 -> 100
Connections:
- net OUT_MINUS: no longer C17.2, C18.2, C19.1, C21.2, C22.2, C25.1, C29.2, D11.2 (A), D20.2 (A), D36.2 (A), D9.1 (K), Q41.2 (B), R89.1, R90.1, T1.4 (SB), T1.5 (SC)
- net at Q41.1 (C): now also Q45.2 (B), R128.2, R129.2, R133.2, R134.2
- new net TRANS1_OUT2: C17.2, C18.2, C19.1, C21.2, C22.2, C25.1, C29.2, D11.2 (A), D20.2 (A), D36.2 (A), D9.1 (K), Q41.2 (B), R89.1, R90.1, T1.4 (SB), T1.5 (SC)
Other:
- moved on the sheet: C34
Changed lines of the file:
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@@
 	)
 	(junction
+		(at 445.77 325.12)
+		(diameter 0)
+		(color 0 0 0 0)
+	)
+	(junction
 		(at 100.33 95.25)
 		(diameter 0)
@@
 	)
 	(junction
-		(at 445.77 309.88)
-		(diameter 0)
-		(color 0 0 0 0)
-	)
-	(junction
 		(at 570.23 287.02)
 		(diameter 0)
@@
 	)
 	(junction
-		(at 407.67 325.12)
-		(diameter 0)
-		(color 0 0 0 0)
-	)
-	(junction
 		(at 684.53 193.04)
 		(diameter 0)
@@
 	)
 	(junction
-		(at 501.65 266.7)
+		(at 407.67 309.88)
 		(diameter 0)
 		(color 0 0 0 0)
 	)
 	(junction
-		(at 422.91 165.1)
+		(at 501.65 266.7)
 		(diameter 0)
 		(color 0 0 0 0)
 	)
 	(junction
-		(at 105.41 165.1)
+		(at 422.91 165.1)
 		(diameter 0)
 		(color 0 0 0 0)
 	)
 	(junction
-		(at 445.77 287.02)
+		(at 105.41 165.1)
 		(diameter 0)
 		(color 0 0 0 0)
@@
 	(wire
 		(pts
+			(xy 407.67 309.88) (xy 429.26 309.88)
+		)
+		(stroke
+			(width 0)
+			(type default)
+		)
+	)
+	(wire
+		(pts
 			(xy 288.29 53.34) (xy 288.29 48.26)
 		)
@@
 	(wire
 		(pts
-			(xy 407.67 287.02) (xy 407.67 325.12)
-		)
-		(stroke
-			(width 0)
-			(type default)
-		)
-	)
-	(wire
-		(pts
 			(xy 191.77 165.1) (xy 191.77 199.39)
 		)
@@
 	(wire
 		(pts
+			(xy 407.67 287.02) (xy 495.3 287.02)
+		)
+		(stroke
+			(width 0)
+			(type default)
+		)
+	)
+	(wire
+		(pts
 			(xy 74.93 300.99) (xy 74.93 309.88)
 		)
@@
 	(wire
 		(pts
-			(xy 252.73 325.12) (xy 407.67 325.12)
+			(xy 252.73 325.12) (xy 445.77 325.12)
 		)
 		(stroke
@@
 	(wire
 		(pts
+			(xy 445.77 325.12) (xy 741.68 325.12)
+		)
+		(stroke
+			(width 0)
+			(type default)
+		)
+	)
+	(wire
+		(pts
 			(xy 317.5 252.73) (xy 317.5 261.62)
 		)
@@
 	(wire
 		(pts
-			(xy 394.97 309.88) (xy 429.26 309.88)
+			(xy 394.97 309.88) (xy 407.67 309.88)
 		)
 		(stroke
@@
 	(wire
 		(pts
+			(xy 407.67 298.45) (xy 407.67 287.02)
+		)
+		(stroke
+			(width 0)
+			(type default)
+		)
+	)
+	(wire
+		(pts
 			(xy 422.91 261.62) (xy 422.91 236.22)
 		)
@@
 	(wire
 		(pts
-			(xy 445.77 246.38) (xy 560.07 246.38)
-		)
-		(stroke
-			(width 0)
-			(type default)
-		)
-	)
-	(wire
-		(pts
 			(xy 707.39 242.57) (xy 707.39 243.84)
 		)
@@
 	(wire
 		(pts
+			(xy 445.77 266.7) (xy 445.77 325.12)
+		)
+		(stroke
+			(width 0)
+			(type default)
+		)
+	)
+	(wire
+		(pts
 			(xy 210.82 90.17) (xy 304.8 90.17)
 		)
@@
 	(wire
 		(pts
-			(xy 445.77 309.88) (xy 482.6 309.88)
-		)
-		(stroke
-			(width 0)
-			(type default)
-		)
-	)
-	(wire
-		(pts
 			(xy 422.91 165.1) (xy 433.07 165.1)
 		)
@@
 	(wire
 		(pts
-			(xy 407.67 325.12) (xy 741.68 325.12)
-		)
-		(stroke
-			(width 0)
-			(type default)
-		)
-	)
-	(wire
-		(pts
 			(xy 546.1 207.01) (xy 556.26 207.01)
 		)
@@
 	(wire
 		(pts
-			(xy 429.26 309.88) (xy 445.77 309.88)
-		)
-		(stroke
-			(width 0)
-			(type default)
-		)
-	)
-	(wire
-		(pts
 			(xy 339.09 124.46) (xy 356.87 124.46)
 		)
@@
 	(wire
 		(pts
-			(xy 445.77 306.07) (xy 445.77 309.88)
+			(xy 407.67 306.07) (xy 407.67 309.88)
 		)
 		(stroke
@@
 	(wire
 		(pts
-			(xy 445.77 287.02) (xy 495.3 287.02)
-		)
-		(stroke
-			(width 0)
-			(type default)
-		)
-	)
-	(wire
-		(pts
 			(xy 304.8 85.09) (xy 306.07 85.09)
 		)
@@
 	(wire
 		(pts
+			(xy 429.26 309.88) (xy 482.6 309.88)
+		)
+		(stroke
+			(width 0)
+			(type default)
+		)
+	)
+	(wire
+		(pts
 			(xy 186.69 48.26) (xy 186.69 53.34)
 		)
@@
 	(wire
 		(pts
-			(xy 407.67 287.02) (xy 445.77 287.02)
-		)
-		(stroke
-			(width 0)
-			(type default)
-		)
-	)
-	(wire
-		(pts
 			(xy 416.56 100.33) (xy 416.56 106.68)
 		)
@@
 	(wire
 		(pts
-			(xy 445.77 287.02) (xy 445.77 298.45)
-		)
-		(stroke
-			(width 0)
-			(type default)
-		)
-	)
-	(wire
-		(pts
-			(xy 434.34 246.38) (xy 438.15 246.38)
+			(xy 434.34 246.38) (xy 560.07 246.38)
 		)
 		(stroke
@@
 	(wire
 		(pts
-			(xy 445.77 266.7) (xy 445.77 287.02)
-		)
-		(stroke
-			(width 0)
-			(type default)
-		)
-	)
-	(wire
-		(pts
 			(xy 416.56 73.66) (xy 416.56 66.04)
 		)
@@
 	(symbol
 		(lib_id "Device:R")
-		(at 441.96 246.38 90)
-		(unit 1)
-		(exclude_from_sim no)
-		(in_bom yes)
-		(on_board yes)
-		(dnp no)
-		(property "Reference" "R114"
-			(at 439.42 243.332 90)
-			(effects
-				(font
-					(size 1.27 1.27)
-				)
-			)
-		)
-		(property "Value" "100"
-			(at 444.754 243.332 90)
-			(effects
-				(font
-					(size 1.27 1.27)
-				)
-			)
-		)
-		(property "Footprint" ""
-			(at 441.96 248.158 90)
-			(effects
-				(font
-					(size 1.27 1.27)
-				)
-				(hide yes)
-			)
-		)
-		(property "Datasheet" "~"
-			(at 441.96 246.38 0)
-			(effects
-				(font
-					(size 1.27 1.27)
-				)
-				(hide yes)
-			)
-		)
-		(property "Description" "Resistor"
-			(at 441.96 246.38 0)
-			(effects
-				(font
-					(size 1.27 1.27)
-				)
-				(hide yes)
-			)
-		)
-		(pin "1"
-		)
-		(pin "2"
-		)
-		(instances
-			(project "PowerSupply"
-				(path "/2ae7299d-2e37-4ad0-914d-1fb9b9570f16"
-					(reference "R114")
-					(unit 1)
-				)
-			)
-		)
-	)
-	(symbol
-		(lib_id "Device:R")
 		(at 725.17 273.05 90)
 		(unit 1)
@@
 	(symbol
 		(lib_id "Device:C_Polarized")
-		(at 445.77 302.26 0)
+		(at 407.67 302.26 0)
 		(unit 1)
 		(exclude_from_sim no)
@@
 		(dnp no)
 		(property "Reference" "C34"
-			(at 447.294 298.704 0)
+			(at 409.194 298.704 0)
 			(effects
 				(font
@@
 		)
 		(property "Value" "100,0 x 10V"
-			(at 447.548 305.308 0)
+			(at 409.448 305.308 0)
 			(effects
 				(font
@@
 		)
 		(property "Footprint" ""
-			(at 446.7352 306.07 0)
+			(at 408.6352 306.07 0)
 			(effects
 				(font
@@
 		)
 		(property "Datasheet" "~"
-			(at 445.77 302.26 0)
+			(at 407.67 302.26 0)
 			(effects
 				(font
@@
 		)
 		(property "Description" "Polarized capacitor"
-			(at 445.77 302.26 0)
+			(at 407.67 302.26 0)
 			(effects
 				(font
@@
 			)
 		)
-		(property "Value" "10"
+		(property "Value" "100"
 			(at 431.8 303.5299 0)
 			(effects
