File: Schematic/PowerSupply.kicad_sch (KiCad schematic)
At the start: 267 parts, among them Q13 BC807, Q14 BC817, Q15 BC807, Q16 BC807, Q17 BC817, Q18 BC807, Q20 BC817, Q21 BC817, Q22 BC807, Q23 BC817, Q24 BC337, Q25 BC328, Q26 BC337, Q27 BC337, Q28 BC337, Q29 BC337, Q30 BC337, Q31 BC328, Q32 BC337, Q33 BC817, Q34 BC817, Q35 BC817, Q36 BC807, Q37 BC807, Q38 BC817, Q39 BC817, Q40 BC807, Q41 BC817, Q42 BC807, Q43 BC807, Q44 BC817, Q45 BC817, Q46 BC817, Q47 BC807, Q48 BC817, Q49 BC817, Q50 BC807, Q51 BC817, Q52 BC807, Q53 BC337, Q54 BC328, Q55 BC337, Q56 BC337, Q57 BC337, Q58 BC337, Q59 BC337, Q60 BC337, Q61 BC337, Q62 BC328, Q63 BC328, Q64 BC337, Q65 BD909, Q66 BD910, Q67 IRLIZ44N, Q68 IRLIZ44N, Q69 BC328, Q70 BC337, Q71 BC337, Q72 BD910, Q73 BC337, Q74 BC337, Q75 BC817, Q76 BC807, Q77 BC817, Q78 BC807, Q79 IRF4905, Q80 IRLIZ44N, Q81 IRF4905, Q82 IRLIZ44N, T2 Transformer_1P_2S, U1 PC817, U2 PC817

Commit message: Add files via upload
Parts:
- removed C1: 1nF x 50V, symbol Device:C
- removed Q14, Q23: BC817, Package_TO_SOT_SMD:SOT-23, symbol Transistor_BJT:BC817
- removed Q22, Q36, Q37: BC807, Package_TO_SOT_SMD:SOT-23, symbol Transistor_BJT:BC807
- removed R28: 4.3K, symbol Device:R
- removed R29, R3, R33: 2.5K, symbol Device:R
- removed R34: 7.5K, symbol Device:R
- removed R5: 100, symbol Device:R
- removed R89: 7.2K, symbol Device:R
- removed U1: PC817, Package_DIP:DIP-4_W7.62mm, symbol Isolator:PC817
- added Q10, Q12, Q7, Q8: BC817, Package_TO_SOT_SMD:SOT-23, symbol Transistor_BJT:BC817
- added Q15, Q16, Q6, Q9: BC807, Package_TO_SOT_SMD:SOT-23, symbol Transistor_BJT:BC807
- added R10, R9: 100, symbol Device:R
- added R12, R137, R14, R15: 3.9K, symbol Device:R
- added R13, R136: 210, symbol Device:R
- added R134: 1.4K, symbol Device:R
- added R138: 15K, symbol Device:R
- added R139, R23, R26, R7, R8: 10K, symbol Device:R
- added R140: 2.2K, symbol Device:R
- added R16: 14K, symbol Device:R
- added R17: 2.4K, symbol Device:R
- added R18, R19: 7.2K, symbol Device:R
- added R2: 1K, symbol Device:R
- R1: renamed from R4; value 15K -> 14K; Conditions (none) -> R=14K, P=0.125W
- R21: renamed from R26; value 4.3K -> 7.2K
- R22: renamed from R36; value 10K -> 7.2K
- R28: renamed from R38; value 10K -> 7.2K
- R30: renamed from R41; value 4.3K -> 7.2K
- R36: renamed from R37; value 2.5K -> 7.5K
- R39: value 2.5K -> 7.5K
- R47: renamed from R92; value 2.5K -> 3.9K
- R58: renamed from R98; value 2.5K -> 15K
- R59: renamed from R95; value 2.5K -> 15K
- R71: renamed from R106; value 2.5K -> 10K
- R72: renamed from R107; value 2.5K -> 10K
- R84: renamed from R108; value 10 -> 100
- R86: renamed from R110; value 10 -> 100
- R88: renamed from R111; value 1K -> 10K
- R89: renamed from R112; value 1K -> 10K
- R94: renamed from R113; value 10 -> 100
- R95: renamed from R115; value 10 -> 100
- R96: renamed from R116; value 1K -> 10K
- R97: renamed from R117; value 1K -> 10K
- renumbered C20 to C1, C45 to C10, C46 to C11, C47 to C12, C48 to C13, C49 to C14, C50 to C15, C51 to C16, C22 to C17, C21 to C18, C52 to C19, C27 to C2, C53 to C20, C23 to C21, C54 to C22, C24 to C23, C25 to C24, C26 to C25, C28 to C26, C29 to C27, C55 to C28, C56 to C29, C38 to C3, C17 to C30, C18 to C31, C19 to C32, C39 to C4, C40 to C5, C41 to C6, C42 to C7, C43 to C8, C44 to C9, D33 to D10, D34 to D11, D35 to D12, D37 to D13, D38 to D14, D14 to D15, D15 to D16, D16 to D17, D17 to D18, D39 to D19, D8 to D20, D12 to D21, D9 to D22, D11 to D23, D41 to D24, D43 to D25, D10 to D26, D44 to D27, D45 to D28, D46 to D29, D13 to D30, D47 to D31, D48 to D32, D25 to D5, D29 to D6, D30 to D7, D31 to D8, D32 to D9, L4 to L1, L5 to L2, L6 to L3, L2 to L4, L1 to L5, Q33 to Q1, Q24 to Q11, Q17 to Q13, Q25 to Q14, Q39 to Q17, Q26 to Q18, Q27 to Q19, Q16 to Q2, Q38 to Q20, Q40 to Q21, Q41 to Q22, Q28 to Q23, Q29 to Q24, Q44 to Q25, Q42 to Q26, Q30 to Q27, Q31 to Q28, Q43 to Q29, Q21 to Q3, Q32 to Q30, Q46 to Q31, Q53 to Q32, Q45 to Q33, Q54 to Q34, Q55 to Q35, Q77 to Q36, Q78 to Q37, Q56 to Q38, Q48 to Q39, Q34 to Q4, Q47 to Q40, Q49 to Q41, Q50 to Q42, Q57 to Q43, Q58 to Q44, Q51 to Q45, Q52 to Q46, Q75 to Q47, Q76 to Q48, Q59 to Q49, Q35 to Q5, Q60 to Q50, Q79 to Q51, Q80 to Q52, Q61 to Q53, Q62 to Q54, Q81 to Q55, Q82 to Q56, Q63 to Q57, Q64 to Q58, Q65 to Q59, Q66 to Q60, Q67 to Q61, Q68 to Q62, Q20 to Q63, Q13 to Q64, Q69 to Q65, Q70 to Q66, Q18 to Q67, Q71 to Q68, Q72 to Q69, Q73 to Q70, Q74 to Q71, Q15 to Q72, R87 to R100, R109 to R101, R114 to R102, R141 to R103, R149 to R104, R150 to R105, R151 to R106, R152 to R107, R153 to R108, R154 to R109, R42 to R11, R155 to R110, R156 to R111, R157 to R112, R158 to R113, R159 to R114, R160 to R115, R161 to R116, R162 to R117, R163 to R118, R164 to R119, R27 to R120, R32 to R121, R165 to R122, R166 to R123, R167 to R124, R168 to R125, R169 to R126, R170 to R127, R171 to R128, R172 to R129, R25 to R130, R30 to R131, R173 to R132, R174 to R133, R31 to R135, R43 to R20, R44 to R24, R45 to R27, R46 to R29, R100 to R3, R47 to R31, R48 to R32, R49 to R33, R50 to R34, R51 to R35, R88 to R37, R40 to R38, R35 to R4, R52 to R40, R53 to R41, R54 to R42, R1 to R43, R2 to R44, R55 to R45, R56 to R46, R97 to R48, R96 to R49, R94 to R5, R57 to R50, R90 to R51, R99 to R52, R58 to R53, R59 to R54, R60 to R55, R61 to R56, R62 to R57, R93 to R6, R63 to R60, R91 to R61, R101 to R62, R64 to R63, R105 to R64, R103 to R65, R65 to R66, R66 to R67, R104 to R68, R102 to R69, R67 to R70, R68 to R73, R69 to R74, R70 to R75, R71 to R76, R72 to R77, R73 to R78, R74 to R79, R75 to R80, R76 to R81, R77 to R82, R78 to R83, R79 to R85, R80 to R87, R81 to R90, R82 to R91, R83 to R92, R84 to R93, R85 to R98, R86 to R99, T2 to T1, U2 to U1
Connections:
- net POWER_IN_24V: now also Q16.2 (E), Q7.3 (C), Q8.3 (C), R14.1, R140.1, R7.1; no longer Q3.3 (C), Q5.3 (C), R21.1, R30.1
- net TRANS1_OUT2: now also R134.2
- net at C1.2, C18.2, C27.2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: now also Q3.2 (E), Q5.2 (E), Q6.3 (C), Q9.3 (C), R138.2, R15.2, R2.2, R8.2; no longer R4.2, R6.2, U1.3
- net at Q13.1 (B), R28.1: now also R23.2
- net at Q17.3 (C), R28.2, R30.2: now also R18.2; no longer Q3.1 (B)
- net at C1.1, Q1.3 (C), Q2.3 (C): now also Q6.1 (B), Q7.1 (B)
- net at Q25.1 (B), R47.2: now also R138.1
- net at Q1.2 (E), R4.1: no longer Q3.2 (E)
- net at Q4.2 (E), R6.1: no longer Q5.2 (E)
- net at Q22.1 (B), R43.2, R44.1: no longer U1.4
- net at Q20.2 (E): now also R137.2; no longer Q21.2 (E)
- net at Q13.3 (C), R21.2, R22.1: now also R19.2; no longer Q5.1 (B)
- net at Q17.1 (B), R22.2: now also R26.2
- net at Q72.1 (B), R135.1: now also R134.1
- net FREQ_CONTROL: no longer names the net of Q1.1 (B), Q4.1 (B), R1.2
- net FREQ_CONTROL: now also R2.1
- new net: R10.1, R12.1, R13.1, R136.1, R137.1, R9.2
- new net: Q12.2 (E), R136.2
- new net: R140.2, R21.1, R30.1
- new net: Q3.1 (B), R18.1
- new net: Q3.3 (C), R4.2
- new net: Q8.2 (E), R9.1
- new net: Q7.2 (E), Q9.1 (B), R8.1
- new net: Q15.2 (E), R13.2
- new net: Q10.3 (C), Q15.1 (B), R14.2, R16.1
- new net: Q6.2 (E), Q8.1 (B), R7.2
- new net: Q9.2 (E), R10.2
- new net: Q5.3 (C), R6.2
- new net: Q10.1 (B), R16.2, R17.1
- new net: Q10.2 (E), Q12.1 (B), R15.1, R17.2
- new net: Q5.1 (B), R19.1
- new net: Q15.3 (C), R23.1
- new net: Q21.2 (E), R12.2
- new net: Q16.1 (B), R139.2
- new net: Q16.3 (C), R26.1
- new net: Q12.3 (C), R139.1
Other:
- note added: "3.4V..4.7V"
- note added: "Ib=0.55mA, i.e. Ik_up_to=18mA"
- note added: "Istab=1.96..4.17mA"
- note added: "On_state: Ikmax_from=1.84mA..3.33mA Ib=0.4..1mA Off_state: Ukmax=4.4V..8V"
- note added: "Ucap"
- note added: "Ucap +/- 0.2"
- note added: "Ucap+[0.5..0.7]"
- note added: "Ucap-[0.5..0.7]"
- note added: "Unorm=16, Umin=13.3V, Umax=24V Imin=3mA Imax=5.5mA"
- note removed: "Power Supply. PWM regulator can be replaced by TL494 like devices. But I wanna to calculate params of device Это блок питания. Но блок питания универсальный. И он еще не доделан и не далеко не все просчитано. Я планирую просчитать номиналы элементов. В данный момент, решил подойти к нему как к тому как проектируют самолеты. В авиации, не применяют сварку по одной простой причине. Нельзя просчитат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"
- moved on the sheet: C1, C10, C11, C12, C13, C14, C15, C16, C17, C18, C19, C2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
